File: PCB/DCDC_3.3.kicad_sch (KiCad schematic)
At the start: 21 parts, among them U10 HT75xx-1-SOT89, U11 LV2842XLVDDCR

Commit message: Minor prod cleanup
Parts:
- renumbered JP6 to JP9
Changed lines of the file:
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@@
         )
         (path "/92dad13e-412a-43d4-9260-9087579302b1/82f027ad-2d00-453d-ab1c-0ba3b5cb1ef7"
-          (reference "C37") (unit 1)
+          (reference "C40") (unit 1)
         )
       )
@@
         )
         (path "/92dad13e-412a-43d4-9260-9087579302b1/82f027ad-2d00-453d-ab1c-0ba3b5cb1ef7"
-          (reference "#PWR090") (unit 1)
+          (reference "#PWR092") (unit 1)
         )
       )
@@
         )
         (path "/92dad13e-412a-43d4-9260-9087579302b1/82f027ad-2d00-453d-ab1c-0ba3b5cb1ef7"
-          (reference "C33") (unit 1)
+          (reference "C36") (unit 1)
         )
       )
@@
         )
         (path "/92dad13e-412a-43d4-9260-9087579302b1/82f027ad-2d00-453d-ab1c-0ba3b5cb1ef7"
-          (reference "C35") (unit 1)
+          (reference "C38") (unit 1)
         )
       )
@@
         )
         (path "/92dad13e-412a-43d4-9260-9087579302b1/82f027ad-2d00-453d-ab1c-0ba3b5cb1ef7"
-          (reference "C34") (unit 1)
+          (reference "C37") (unit 1)
         )
       )
@@
         )
         (path "/92dad13e-412a-43d4-9260-9087579302b1/82f027ad-2d00-453d-ab1c-0ba3b5cb1ef7"
-          (reference "C38") (unit 1)
+          (reference "C41") (unit 1)
         )
       )
@@
         )
         (path "/92dad13e-412a-43d4-9260-9087579302b1/82f027ad-2d00-453d-ab1c-0ba3b5cb1ef7"
-          (reference "#PWR091") (unit 1)
+          (reference "#PWR093") (unit 1)
         )
       )
@@
         )
         (path "/92dad13e-412a-43d4-9260-9087579302b1/82f027ad-2d00-453d-ab1c-0ba3b5cb1ef7"
-          (reference "#PWR095") (unit 1)
+          (reference "#PWR097") (unit 1)
         )
       )
@@
         )
         (path "/92dad13e-412a-43d4-9260-9087579302b1/82f027ad-2d00-453d-ab1c-0ba3b5cb1ef7"
-          (reference "C36") (unit 1)
+          (reference "C39") (unit 1)
         )
       )
@@
         )
         (path "/92dad13e-412a-43d4-9260-9087579302b1/82f027ad-2d00-453d-ab1c-0ba3b5cb1ef7"
-          (reference "#PWR093") (unit 1)
+          (reference "#PWR095") (unit 1)
         )
       )
@@
         )
         (path "/92dad13e-412a-43d4-9260-9087579302b1/82f027ad-2d00-453d-ab1c-0ba3b5cb1ef7"
-          (reference "#PWR092") (unit 1)
+          (reference "#PWR094") (unit 1)
         )
       )
@@
         )
         (path "/92dad13e-412a-43d4-9260-9087579302b1/82f027ad-2d00-453d-ab1c-0ba3b5cb1ef7"
-          (reference "#PWR094") (unit 1)
+          (reference "#PWR096") (unit 1)
         )
       )
@@
         )
         (path "/92dad13e-412a-43d4-9260-9087579302b1/82f027ad-2d00-453d-ab1c-0ba3b5cb1ef7"
-          (reference "#PWR096") (unit 1)
+          (reference "#PWR098") (unit 1)
         )
       )
@@
         )
         (path "/92dad13e-412a-43d4-9260-9087579302b1/82f027ad-2d00-453d-ab1c-0ba3b5cb1ef7"
-          (reference "#PWR089") (unit 1)
+          (reference "#PWR091") (unit 1)
         )
       )
@@
         )
         (path "/92dad13e-412a-43d4-9260-9087579302b1/82f027ad-2d00-453d-ab1c-0ba3b5cb1ef7"
-          (reference "#PWR097") (unit 1)
+          (reference "#PWR099") (unit 1)
         )
       )
@@
         )
         (path "/92dad13e-412a-43d4-9260-9087579302b1/82f027ad-2d00-453d-ab1c-0ba3b5cb1ef7"
-          (reference "#PWR088") (unit 1)
+          (reference "#PWR090") (unit 1)
         )
       )
@@
   (symbol (lib_id "Device:R") (at 105.664 54.61 180) (unit 1)
     (in_bom no) (on_board yes) (dnp yes)
-    (property "Reference" "JP6" (at 103.886 55.88 0)
+    (property "Reference" "JP9" (at 103.886 55.88 0)
       (effects (font (size 1.27 1.27)) (justify left))
     )
@@
       (project "StepperServoCAN"
         (path "/92dad13e-412a-43d4-9260-9087579302b1/82f027ad-2d00-453d-ab1c-0ba3b5cb1ef7"
-          (reference "JP6") (unit 1)
-        )
-      )
+          (reference "JP9") (unit 1)
+        )
+      )
